Commit message: Update: urdf without stl

File: basic_mobile_robot/models/basic_mobile_bot_v1.urdf (robot description, URDF)
Before this commit: robot basic_mobile_bot, 7 links, 6 joints
Links:
- link base_link: geometry collision box size=0.7 0.39 0.2; visual box size=0.70 0.15 0.40

File: basic_mobile_robot/models/basic_mobile_bot_v1.urdf.xacro (robot description, xacro)
@@ -54,5 +54,5 @@
       <origin xyz="0 0 -0.05" rpy="1.5707963267949 0 3.141592654" />
       <geometry>
-        <mesh filename="package://basic_mobile_robot/meshes/robot_base.stl" />
+        <box size="0.70 0.15 0.40" />
       </geometry>
       <material name="Red">
